File: rda5708m.sch (EAGLE design)
At the start: 36 parts, among them IC1 RDA5807M, IC2 STM32L052K8U, Q1 32768Hz, U2 TPS73033, U3 MCP73831

Commit message: fabricated version
Parts:
- removed C8: 2.2uF, microbuilder:CAP_CERAMIC0805
- removed SW1: (no value), microbuilder:SWITCH_SPST
- added CN1: (no value), rda5807m:AUDIO_3.5JACK
- added Q3: IRLML5203, microbuilder:MOSFET-P
- added Q4: (no value), microbuilder:MOSFET-NREFLOW
- added R10: 200k, microbuilder:RESISTOR0603
- added R8, R9: 10k, microbuilder:RESISTOR0603
- added S4: (no value), rda5807m:SWITCH-SPDTPTH2
- added TP1, TP2: TPTP10R, testpad:TPTP10R
- BT1: device SparkFun-Batteries:BATTERY-6.8MM_SMD -> rda5807m:BATTERY
- C1, C10, C11, C15, C2, C3, C4, C5, C6, C7, C9: device microbuilder:CAP_CERAMIC0805 -> microbuilder:CAP_CERAMIC0603
- Q1: device crystal:CRYSTALTC26H -> rda5807m:CRYSTAL
- R1, R2, R3, R4, R5, R6, R7: device microbuilder:RESISTOR0805 -> microbuilder:RESISTOR0603
- S1, S2, S3: device SparkFun-Retired:TAC_SWITCHSMD -> rda5807m:TAC_SWITCH
- U1: device microbuilder:DISP_OLED_UG-2864HSWEG010.96" -> rda5807m:DISP_OLED_UG-2864HSWEG012SIDE
- U3: device SparkFun-IC-Power:MCP73831 -> rda5807m:MCP73831
- USB1: device con-hirose:MICRO-USB-SHIELD-MICRO_USB-B_4.85_HORN -> rda5807m:MICRO-USB-SHIELD-MICRO_USB-B_4.85_HORN
Connections:
- net N$19 renamed SPI_DC
- net N$2 renamed VUSB
- net N$20 renamed SPI_SCK
- net N$21 renamed SPI_MOSI
- removed net 5.0V: C14.P$2, C15.P$2, R4.1, SW1.S, U2.EN, U2.IN
- new net +5V: C14.P$2, C15.P$2, S4.P, U2.EN, U2.IN
- new net N$18: Q3.G, Q4.D, R10.2
- new net N$19: IC2MCU.PA3
- new net N$2: Q3.D, R4.1
- new net N$20: IC2MCU.PA2
- new net N$21: IC2MCU.PA1
- new net N$25: C13.P$2, CN1.P$3
- new net N$26: C12.P$2, CN1.P$2
- new net N$27: IC2MCU.PA0
- new net N$29: IC2MCU.PB2
- new net PA10: IC2MCU.PA10, Q4.G
- new net PA8: IC2MCU.PA8, U3.STAT
- new net PA9: IC2MCU.PA9
- new net PC15: IC2MCU.PC15-OSC_OUT
- new net SCLK: IC1.SCLK, IC2MCU.PB6, R2.1
- new net SDIO: IC1.SDIO, IC2MCU.PB7, R9.1
- new net SWCLK: IC2MCU.PA14, TP1.TP
- new net SWDIO: IC2MCU.PA13, TP2.TP
- new net VBAT: BT1.+, Q2.D, Q3.S, R10.1, U3.VBAT
- net 3.3V: now also R2.2, R8.1, R9.2; no longer C8.P$2, R2.1
- net GND: now also CN1.P$1, Q4.S; no longer C8.P$1
- net N$11: now also IC2MCU.PA15; no longer IC1.SCLK, IC2MCU.PB6
- net N$15: now also S4.O; no longer SW1.P
- net N$16: now also IC2MCU.PA4; no longer BT1.+, Q2.D, U3.VBAT
- net N$4: now also IC2MCU.PB8; no longer IC1.SDIO, IC2MCU.PB7
- net PC14: no longer U3.STAT
- net RST: now also R8.2; no longer R2.2
Other:
- moved on the sheet: C14, C15, C3, C4, D1, Q2, R2, R4, R5, R6, R7, S1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

Commit message: fabricated release
Parts:
- removed IC1: RDA5807M, rda5807m:RDA5807M
- added OLED: (no value), rda5807m:DISP_OLED_UG-2864HSWEG012SIDE
- U1: value (none) -> MCP73831; device rda5807m:DISP_OLED_UG-2864HSWEG012SIDE -> rda5807m:MCP73831
- U3: value MCP73831 -> RDA5807M; device rda5807m:MCP73831 -> rda5807m:RDA5807M
- renumbered IC2 to U4, Q1 to Z1, Q2 to T3, Q3 to T1, Q4 to T2, TP1 to SWCLK, TP2 to SWDIO, USB1 to USB
Connections:
- new net N$28: U3.FMIN
- net 3.3V: now also OLED.VBAT, OLED.VDD, U3.VDD; no longer IC1.VDD, U1.VBAT, U1.VDD
- net GND: now also OLED.BS0, OLED.BS1, OLED.BS2, OLED.NC(GND)@1, OLED.NC(GND)@2, OLED.VLSS, OLED.VSS, U3.GND, U3.GND@1, U3.GND@2; no longer IC1.GND, IC1.GND@1, IC1.GND@2, U1.BS0, U1.BS1, U1.BS2, U1.NC(GND)@1, U1.NC(GND)@2, U1.VLSS, U3.VSS
- net N$1: now also U3.RCLK; no longer IC1.RCLK
- net N$10: now also U3.ROUT; no longer IC1.ROUT
- net N$14: now also U1.PROG; no longer U3.PROG
- net N$17: now also OLED./CS; no longer U1./CS
- net N$22: now also OLED.IREF; no longer U1.IREF
- net N$23: now also OLED.VCOMH; no longer U1.VCOMH
- net N$24: now also OLED.VCC; no longer U1.VCC
- net N$5: now also U3.LOUT; no longer IC1.LOUT
- net N$6: now also OLED.C2P; no longer U1.C2P
- net N$7: now also OLED.C2N; no longer U1.C2N
- net N$8: now also OLED.C1P; no longer U1.C1P
- net N$9: now also OLED.C1N; no longer U1.C1N
- net PA8: now also U1.STAT; no longer U3.STAT
- net RST: now also OLED./RES; no longer U1./RES
- net SCLK: now also U3.SCLK; no longer IC1.SCLK
- net SDIO: now also U3.SDIO; no longer IC1.SDIO
- net SPI_DC: now also OLED.DC/I2C_SA0; no longer U1.DC/I2C_SA0
- net SPI_MOSI: now also OLED.D1/SPI_SDIN/I2C_SDA; no longer U1.D1/SPI_SDIN/I2C_SDA
- net SPI_SCK: now also OLED.D0/SPI_SCLK/I2C_SCK; no longer U1.D0/SPI_SCLK/I2C_SCK
- net VBAT: now also U1.VBAT; no longer U3.VBAT
- net VUSB: now also U1.VIN; no longer U3.VIN

Commit message: pcb fix
Connections:
- net N$11 renamed PA15
- net N$12 renamed PA11
- net N$13 renamed PA12
- net N$16 renamed PA4
- net N$17 renamed PB1
- net N$19 renamed PA3
- net N$20 renamed PA2
- net N$21 renamed PA1
- net N$27 renamed PA0
- net N$28 renamed ANT
- net N$29 renamed PB2
- net N$3 renamed BOOT0
- net N$4 renamed PB8
Changed lines of the file:
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@@
 </segment>
 </net>
-<net name="N$3" class="0">
+<net name="BOOT0" class="0">
 <segment>
 <pinref part="U4" gate="MCU" pin="BOOT0"/>
@@
 </segment>
 </net>
-<net name="N$17" class="0">
+<net name="PB1" class="0">
 <segment>
 <pinref part="OLED" gate="G$1" pin="/CS"/>
@@
 </segment>
 </net>
-<net name="N$12" class="0">
+<net name="PA11" class="0">
 <segment>
 <wire x1="99.06" y1="114.3" x2="71.12" y2="114.3" width="0.1524" layer="91"/>
@@
 </segment>
 </net>
-<net name="N$13" class="0">
+<net name="PA12" class="0">
 <segment>
 <wire x1="99.06" y1="111.76" x2="73.66" y2="111.76" width="0.1524" layer="91"/>
@@
 </segment>
 </net>
-<net name="N$29" class="0">
+<net name="PB2" class="0">
 <segment>
 <pinref part="U4" gate="MCU" pin="PB2"/>
@@
 </segment>
 </net>
-<net name="N$4" class="0">
+<net name="PB8" class="0">
 <segment>
 <pinref part="U4" gate="MCU" pin="PB8"/>
@@
 </segment>
 </net>
-<net name="N$11" class="0">
+<net name="PA15" class="0">
 <segment>
 <pinref part="U4" gate="MCU" pin="PA15"/>
@@
 </segment>
 </net>
-<net name="N$16" class="0">
+<net name="PA4" class="0">
 <segment>
 <pinref part="U4" gate="MCU" pin="PA4"/>
@@
 </segment>
 </net>
-<net name="N$19" class="0">
+<net name="PA3" class="0">
 <segment>
 <pinref part="U4" gate="MCU" pin="PA3"/>
@@
 </segment>
 </net>
-<net name="N$20" class="0">
+<net name="PA2" class="0">
 <segment>
 <pinref part="U4" gate="MCU" pin="PA2"/>
@@
 </segment>
 </net>
-<net name="N$21" class="0">
+<net name="PA1" class="0">
 <segment>
 <pinref part="U4" gate="MCU" pin="PA1"/>
@@
 </segment>
 </net>
-<net name="N$27" class="0">
+<net name="PA0" class="0">
 <segment>
 <pinref part="U4" gate="MCU" pin="PA0"/>
@@
 </segment>
 </net>
-<net name="N$28" class="0">
+<net name="ANT" class="0">
 <segment>
 <pinref part="U3" gate="G$1" pin="FMIN"/>
